Commit message: got ardrone_crash_bumper working

File: cvg_sim_gazebo/urdf/quadrotor_base.urdf.xacro (robot description, xacro)
@@ -27,4 +27,15 @@
     <gazebo reference="base_link">
       <turnGravityOff>false</turnGravityOff>
+      <sensor name="base_contact" type="contact" update_rate="10.0">
+        <contact>
+          <collision>base_link_collision</collision>
+        </contact>
+        <plugin name="bumper" filename="libgazebo_ros_bumper.so">
+          <alwaysOn>true</alwaysOn>
+          <updateRate>50.0</updateRate>
+          <frameName>world</frameName>
+          <bumperTopicName>ardrone_crash_bumper</bumperTopicName>
+        </plugin>
+      </sensor>
     </gazebo>
     <!-- Gazebo Plugins -->

File: cvg_sim_gazebo/urdf/quadrotor_sensors.urdf.xacro (robot description, xacro)
@@ -22,11 +22,13 @@
     <!-- Forward facing camera -->
     <xacro:include filename="$(find cvg_sim_gazebo)/urdf/sensors/generic_camera.urdf.xacro" />
-    <xacro:generic_camera name="front" sim_name="ardrone" parent="base_link" update_rate="60" res_x="640" res_y="360" image_format="R8G8B8" hfov="${81*M_PI/180}">
+    <!--<xacro:generic_camera name="front" sim_name="ardrone" parent="base_link" update_rate="10" res_x="64" res_y="36" image_format="R8G8B8" hfov="${81*M_PI/180}">-->
+    <!--<xacro:generic_camera name="front" sim_name="ardrone" parent="base_link" update_rate="10" res_x="32" res_y="18" image_format="R8G8B8" hfov="${81*M_PI/180}">-->
+    <xacro:generic_camera name="front" sim_name="ardrone" parent="base_link" update_rate="400" res_x="32" res_y="18" image_format="L8" hfov="${81*M_PI/180}">
       <origin xyz="0.21 0.0 0.01" rpy="0 0 0"/>
     </xacro:generic_camera>
     <!-- Downward facing camera -->
-    <xacro:include filename="$(find cvg_sim_gazebo)/urdf/sensors/generic_camera.urdf.xacro" />
-    <xacro:generic_camera name="bottom" sim_name="ardrone" parent="base_link" update_rate="60" res_x="640" res_y="360" image_format="R8G8B8" hfov="${81*M_PI/180}">
-        <origin xyz="0.15 0.0 0.0" rpy="0 ${M_PI/2} 0"/>
-    </xacro:generic_camera>
+    <!--<xacro:include filename="$(find cvg_sim_gazebo)/urdf/sensors/generic_camera.urdf.xacro" />-->
+    <!--<xacro:generic_camera name="bottom" sim_name="ardrone" parent="base_link" update_rate="60" res_x="640" res_y="360" image_format="R8G8B8" hfov="${81*M_PI/180}">-->
+      <!--<origin xyz="0.15 0.0 0.0" rpy="0 ${M_PI/2} 0"/>-->
+    <!--</xacro:generic_camera>-->
 </robot>
